Commit message: add faked aligned color to depth camera model which simply changes the color image intrinsics and extrinsics to exactly match the depth

File: realsense2_description/urdf/_d435_aligned_colortodepth.gazebo.xacro (robot description, xacro)
@@ -25,8 +25,8 @@
       <sensor name="${camera_name}color" type="camera">
         <camera name="${camera_name}">
-          <horizontal_fov>${69.4*deg_to_rad}</horizontal_fov>
+          <horizontal_fov>${85.2*deg_to_rad}</horizontal_fov> <!-- 69.4*deg_to_rad -->
           <image>
-            <width>640</width>
-            <height>480</height>
+            <width>1280</width>  <!-- 640 -->
+            <height>720</height> <!-- 480 -->
             <format>RGB_INT8</format>
           </image>

File: realsense2_description/urdf/_d435_aligned_colortodepth.urdf.xacro (robot description, xacro)
@@ -8,5 +8,5 @@
 <robot name="sensor_d435" xmlns:xacro="http://ros.org/wiki/xacro">
   <!-- Includes -->
-  <xacro:include filename="$(find realsense2_description)/urdf/_d435.gazebo.xacro" />
+  <xacro:include filename="$(find realsense2_description)/urdf/_d435_aligned_colortodepth.gazebo.xacro" />
   <xacro:include filename="$(find realsense2_description)/urdf/_materials.urdf.xacro" />
   <xacro:include filename="$(find realsense2_description)/urdf/_usb_plug.urdf.xacro" />
@@ -17,5 +17,5 @@
     <xacro:property name="d435_cam_depth_to_infra1_offset" value="0.0"/>
     <xacro:property name="d435_cam_depth_to_infra2_offset" value="-0.050"/>
-    <xacro:property name="d435_cam_depth_to_color_offset" value="0.015"/>
+    <xacro:property name="d435_cam_depth_to_color_offset" value="0.0"/> <!-- 0.015 -->
     <!-- The following values model the aluminum peripherial case for the
   	D435 camera, with the camera joint represented by the actual

File: realsense2_description/urdf/test_d435_camera_aligned_colortodepth.urdf.xacro (robot description, xacro)
@@ -7,5 +7,5 @@
   <xacro:arg name="topics_ns" default="camera" />
   <xacro:arg name="publish_pointcloud" default="false" />
-  <xacro:include filename="$(find realsense2_description)/urdf/_d435.urdf.xacro" />
+  <xacro:include filename="$(find realsense2_description)/urdf/_d435_aligned_colortodepth.urdf.xacro" />
   <xacro:arg name="cam_x"           default="0"     doc="How far forward to place the base of the robot in [m]?" />
   <xacro:arg name="cam_y"           default="0"     doc="How far leftwards to place the base of the robot in [m]?" />
@@ -14,5 +14,5 @@
   <xacro:arg name="cam_pitch"       default="0"     doc="How much to rotate the base of the robot around its Y-axis in [rad]?" />
   <xacro:arg name="cam_yaw"         default="0"     doc="How much to rotate the base of the robot around its Z-axis in [rad]?" />
-  <xacro:arg name="fps"       default="30"     doc="Frame rate of depth image" />
+  <xacro:arg name="fps"       default="30"     doc="Frame rate of depth and color image" />
   <link name="world" />
   <xacro:sensor_d435 parent="world" use_nominal_extrinsics="$(arg use_nominal_extrinsics)" add_plug="$(arg add_plug)" use_mesh="$(arg use_mesh)" name="$(arg name)" topics_ns="$(arg topics_ns)" fps="$(arg fps)" publish_pointcloud="$(arg publish_pointcloud)">
