Commit message: add usage of yaml file from extrinsic calibration to the d455 urdf

File: realsense2_description/urdf/test_d455_camera_aligned_depthtocolor.urdf.xacro (robot description, xacro)
@@ -7,14 +7,16 @@
   <xacro:arg name="publish_pointcloud" default="false" />
   <xacro:include filename="$(find realsense2_description)/urdf/_d455_aligned_depthtocolor.urdf.xacro" />
-  <xacro:arg name="cam_x"           default="0"     doc="How far forward to place the base of the robot in [m]?" />
-  <xacro:arg name="cam_y"           default="0"     doc="How far leftwards to place the base of the robot in [m]?" />
-  <xacro:arg name="cam_z"           default="0"     doc="How far upwards to place the base of the robot in [m]?" />
-  <xacro:arg name="cam_roll"        default="0"     doc="How much to rotate the base of the robot around its X-axis in [rad]?" />
-  <xacro:arg name="cam_pitch"       default="0"     doc="How much to rotate the base of the robot around its Y-axis in [rad]?" />
-  <xacro:arg name="cam_yaw"         default="0"     doc="How much to rotate the base of the robot around its Z-axis in [rad]?" />
+  <xacro:property name="yaml_file" value="$(find screwing_simulation)/config/cam_pose.yaml" />
+  <xacro:property name="cam_pose" value="${load_yaml(yaml_file)}"/>
+  <xacro:property name="cam_x"           value="${cam_pose['x']}"     doc="How far forward to place the base of the robot in [m]?" />
+  <xacro:property name="cam_y"           value="${cam_pose['y']}"     doc="How far leftwards to place the base of the robot in [m]?" />
+  <xacro:property name="cam_z"           value="${cam_pose['z']}"     doc="How far upwards to place the base of the robot in [m]?" />
+  <xacro:property name="cam_roll"        value="${cam_pose['roll']}"     doc="How much to rotate the base of the robot around its X-axis in [rad]?" />
+  <xacro:property name="cam_pitch"       value="${cam_pose['pitch']}"     doc="How much to rotate the base of the robot around its Y-axis in [rad]?" />
+  <xacro:property name="cam_yaw"         value="${cam_pose['yaw']}"     doc="How much to rotate the base of the robot around its Z-axis in [rad]?" />
   <xacro:arg name="fps"       default="30"     doc="Frame rate of depth and color image" />
   <link name="world" />
   <xacro:sensor_d455 parent="world" use_nominal_extrinsics="$(arg use_nominal_extrinsics)" add_plug="$(arg add_plug)" name="$(arg name)" topics_ns="$(arg topics_ns)" fps="$(arg fps)" publish_pointcloud="$(arg publish_pointcloud)">
-    <origin xyz="$(arg cam_x) $(arg cam_y) $(arg cam_z)" rpy="$(arg cam_roll) $(arg cam_pitch) $(arg cam_yaw)"/>
+    <origin xyz="${cam_x} ${cam_y} ${cam_z}" rpy="${cam_roll} ${cam_pitch} ${cam_yaw}"/>
   </xacro:sensor_d455>
 </robot>
