Commit message: add actual optical frame used by gazebo in the d455 aligned depth to color model

File: realsense2_description/urdf/_d435_aligned_colortodepth.urdf.xacro (robot description, xacro)
@@ -17,5 +17,5 @@
     <xacro:property name="d435_cam_depth_to_infra1_offset" value="0.0"/>
     <xacro:property name="d435_cam_depth_to_infra2_offset" value="-0.050"/>
-    <xacro:property name="d435_cam_depth_to_color_offset" value="0.0"/> <!-- 0.015 -->
+    <xacro:property name="d435_cam_depth_to_color_offset" value="0.0"/>  <!-- changed this to 0 to align color to depth--> <!-- 0.015 -->
     <!-- The following values model the aluminum peripherial case for the
   	D435 camera, with the camera joint represented by the actual

File: realsense2_description/urdf/_d455_aligned_depthtocolor.urdf.xacro (robot description, xacro)
@@ -76,4 +76,10 @@
     <xacro:if value="${use_nominal_extrinsics}">
       <!-- camera depth joints and links -->
+      <joint name="${name}_optical_joint" type="fixed">
+        <origin xyz="0 0 0" rpy="${-M_PI/2} 0 ${-M_PI/2}" />
+        <parent link="${name}_link" />
+        <child link="${name}_optical_frame" />
+      </joint>
+      <link name="${name}_optical_frame"/>
       <joint name="${name}_depth_joint" type="fixed">
         <origin xyz="0 ${d455_cam_depth_to_color_offset} 0" rpy="0 0 0"/> <!-- added offset here to match depth to color frame (originally xyz = 0,0,0)-->

File: realsense2_description/urdf/test_d435_camera_aligned_colortodepth.urdf.xacro (robot description, xacro)
@@ -8,14 +8,23 @@
   <xacro:arg name="publish_pointcloud" default="false" />
   <xacro:include filename="$(find realsense2_description)/urdf/_d435_aligned_colortodepth.urdf.xacro" />
-  <xacro:arg name="cam_x"           default="0"     doc="How far forward to place the base of the robot in [m]?" />
+  <xacro:property name="yaml_file" value="$(find screwing_simulation)/config/cam_pose.yaml" />
+  <xacro:property name="cam_pose" value="${load_yaml(yaml_file)}"/>
+  <xacro:property name="cam_x"           value="${cam_pose['x']}"     doc="How far forward to place the base of the robot in [m]?" />
+  <xacro:property name="cam_y"           value="${cam_pose['y']}"     doc="How far leftwards to place the base of the robot in [m]?" />
+  <xacro:property name="cam_z"           value="${cam_pose['z']}"     doc="How far upwards to place the base of the robot in [m]?" />
+  <xacro:property name="cam_roll"        value="${cam_pose['roll']}"     doc="How much to rotate the base of the robot around its X-axis in [rad]?" />
+  <xacro:property name="cam_pitch"       value="${cam_pose['pitch']}"     doc="How much to rotate the base of the robot around its Y-axis in [rad]?" />
+  <xacro:property name="cam_yaw"         value="${cam_pose['yaw']}"     doc="How much to rotate the base of the robot around its Z-axis in [rad]?" />
+  <!-- <xacro:arg name="cam_x"           default="0"     doc="How far forward to place the base of the robot in [m]?" />
   <xacro:arg name="cam_y"           default="0"     doc="How far leftwards to place the base of the robot in [m]?" />
   <xacro:arg name="cam_z"           default="0"     doc="How far upwards to place the base of the robot in [m]?" />
   <xacro:arg name="cam_roll"        default="0"     doc="How much to rotate the base of the robot around its X-axis in [rad]?" />
   <xacro:arg name="cam_pitch"       default="0"     doc="How much to rotate the base of the robot around its Y-axis in [rad]?" />
-  <xacro:arg name="cam_yaw"         default="0"     doc="How much to rotate the base of the robot around its Z-axis in [rad]?" />
+  <xacro:arg name="cam_yaw"         default="0"     doc="How much to rotate the base of the robot around its Z-axis in [rad]?" /> -->
   <xacro:arg name="fps"       default="30"     doc="Frame rate of depth and color image" />
   <link name="world" />
   <xacro:sensor_d435 parent="world" use_nominal_extrinsics="$(arg use_nominal_extrinsics)" add_plug="$(arg add_plug)" use_mesh="$(arg use_mesh)" name="$(arg name)" topics_ns="$(arg topics_ns)" fps="$(arg fps)" publish_pointcloud="$(arg publish_pointcloud)">
-    <origin xyz="$(arg cam_x) $(arg cam_y) $(arg cam_z)" rpy="$(arg cam_roll) $(arg cam_pitch) $(arg cam_yaw)"/>
+    <!-- <origin xyz="$(arg cam_x) $(arg cam_y) $(arg cam_z)" rpy="$(arg cam_roll) $(arg cam_pitch) $(arg cam_yaw)"/> -->
+    <origin xyz="${cam_x} ${cam_y} ${cam_z}" rpy="${cam_roll} ${cam_pitch} ${cam_yaw}"/>
   </xacro:sensor_d435>
 </robot>
