Commit message: add hack to allow camera to float and to be able to specify changes in pose freely

File: realsense2_description/urdf/_d455_aligned_depthtocolor.gazebo.xacro (robot description, xacro)
@@ -119,6 +119,6 @@
         <colorUpdateRate>0.0</colorUpdateRate> <!-- 30 -->
         <infraredUpdateRate>0.0</infraredUpdateRate> <!-- 30 -->
-        <depthTopicName>depth/image_raw</depthTopicName>
-        <depthCameraInfoTopicName>depth/camera_info</depthCameraInfoTopicName>
+        <depthTopicName>aligned_depth_to_color/image_raw</depthTopicName>
+        <depthCameraInfoTopicName>aligned_depth_to_color/camera_info</depthCameraInfoTopicName>
         <colorTopicName>color/image_raw</colorTopicName>
         <colorCameraInfoTopicName>color/camera_info</colorCameraInfoTopicName>

File: realsense2_description/urdf/test_d455_camera_aligned_depthtocolor.urdf.xacro (robot description, xacro)
@@ -6,13 +6,14 @@
   <xacro:arg name="topics_ns" default="camera" />
   <xacro:arg name="publish_pointcloud" default="false" />
+  <xacro:arg name="cam_pose_config" default="$(find contact_simulation)/config/cam_pose.yaml" />
   <xacro:include filename="$(find realsense2_description)/urdf/_d455_aligned_depthtocolor.urdf.xacro" />
-  <xacro:property name="yaml_file" value="$(find screwing_simulation)/config/cam_pose.yaml" />
-  <xacro:property name="cam_pose" value="${load_yaml(yaml_file)}"/>
-  <xacro:property name="cam_x"           value="${cam_pose['x']}"     doc="How far forward to place the base of the robot in [m]?" />
-  <xacro:property name="cam_y"           value="${cam_pose['y']}"     doc="How far leftwards to place the base of the robot in [m]?" />
-  <xacro:property name="cam_z"           value="${cam_pose['z']}"     doc="How far upwards to place the base of the robot in [m]?" />
-  <xacro:property name="cam_roll"        value="${cam_pose['roll']}"     doc="How much to rotate the base of the robot around its X-axis in [rad]?" />
-  <xacro:property name="cam_pitch"       value="${cam_pose['pitch']}"     doc="How much to rotate the base of the robot around its Y-axis in [rad]?" />
-  <xacro:property name="cam_yaw"         value="${cam_pose['yaw']}"     doc="How much to rotate the base of the robot around its Z-axis in [rad]?" />
+  <xacro:property name="yaml_file" value="$(arg cam_pose_config)" />
+  <xacro:property name="cam_pose" value="${xacro.load_yaml(yaml_file)}"/>
+  <xacro:property name="cam_x" value="${cam_pose['x']}" />
+  <xacro:property name="cam_y" value="${cam_pose['y']}" />
+  <xacro:property name="cam_z" value="${cam_pose['z']}" />
+  <xacro:property name="cam_roll" value="${cam_pose['roll']}"  />
+  <xacro:property name="cam_pitch" value="${cam_pose['pitch']}" />
+  <xacro:property name="cam_yaw" value="${cam_pose['yaw']}"   />
   <xacro:arg name="fps"       default="30"     doc="Frame rate of depth and color image" />
   <link name="world" />
